File: cruise/cruise.sch (EAGLE design)
At the start: 26 parts, among them IC1 24C04ASM, U1 STM32F103CBT6

Commit message: работа над схемой
Parts:
- removed T3: (no value), transistor:MMBT4401LT1-NPN-SOT23-BEC
- added C10, C9: 20pf, rcl:C-EUC0805
- added C11, C12, C14, C16, C17, C18, C19: 100nf, rcl:C-EUC0805
- added C13: 1uF, rcl:C-EUC0805
- added C15: 10uF, rcl:C-EUC0805
- added C5, C7: 10uF, rcl:CPOL-EUCT6032
- added C6, C8: 1uF, rcl:CPOL-EUCT6032
- added D1, D2: 5.1V, diode:ZENER-DIODESOD80C
- added D3, D5, D6: 3V3, diode:ZENER-DIODESOD80C
- added D4: 3v3, diode:ZENER-DIODESOD80C
- added D7, D8: 3.3V, diode:ZENER-DIODESOD80C
- added J1: (no value), jumper:J2X2MM
- added M0, M1, PAD1, PAD2, PAD3, PAD4, PAD5: (no value), wirepad:2,54/1,0
- added Q1, Q2, Q3: BSS138, m-pad-2.1:BSS138
- added Q4: 8MHz, crystal:CRYSTALSM49
- added R18: 200, resistor:R-EU_R0805
- added R19: 1.5K, resistor:R-EU_R0805
- added R20, R22, R23, R24, R27: 10K, resistor:R-EU_R0805
- added R21: 6.8K, resistor:R-EU_R0805
- added R25, R26: 4.7K, resistor:R-EU_R0805
- added S1: RESET_BUTTON, m-pad-2.1:RESET_BUTTON
- added X1: JST-XH-02-PIN-LONG-PAD, Rembrandt Electronics - JST XH Connectors v1-0:JST-XH-02-PIN-LONG-PAD
- added X2: JST-XH-04-PIN-LONG-PAD, Rembrandt Electronics - JST XH Connectors v1-0:JST-XH-04-PIN-LONG-PAD
- added X3: JST-XH-05-PIN-LONG-PAD, Rembrandt Electronics - JST XH Connectors v1-0:JST-XH-05-PIN-LONG-PAD
- added X4: JST-XH-06-PIN-LONG-PAD, Rembrandt Electronics - JST XH Connectors v1-0:JST-XH-06-PIN-LONG-PAD
- C1: value 1nf -> 1nF; device rcl:C-EUC1206 -> rcl:C-EUC0805
- C2: value 10uf -> 1nF; device rcl:CPOL-EUB/3528-21W -> rcl:C-EUC0805
- C3: value 1nf -> 5uF; device rcl:C-EUC1206 -> rcl:CPOL-EUCT6032
- C4: value 10uf -> 10uF; device rcl:CPOL-EUB/3528-21W -> rcl:CPOL-EUCT6032
- R1: value 10k -> 10K
- R10, R2: value 6.8k -> 10K
- R11, R7, R9: value 10k -> 3.3K
- R12, R14, R16: value 4.7k -> 10K
- R13: value 4.7k -> 3.3K
- R15, R17: value 4.7k -> 6.8K
- R3, R5: value 10k -> 4.7K
- R4: value 6.8k -> 4.7K
- R6, R8: value 3.3k -> 10K
- T1, T2: device transistor:MMBT4401LT1-NPN-SOT23-BEC -> transistor-neu-to92:MMBT4401LT1-NPN-SOT23-BEC
Connections:
- net SWDCLK renamed N$40
- net SWDIO renamed N$39
- net USART_RX renamed N$36
- net USART_TX renamed N$34
- net USB_CTS renamed N$37
- net USB_RTS renamed N$38
- removed net I2C_SCL: U1.PB6
- removed net I2C_SDA: U1.PB7
- removed net STOP_EXTI3: R14.1, R7.1, R8.2, T2.B, T2.C, U1.PA3
- removed net VNH2_SP30_CS_IN: R9.2
- new net +12V: X2-3.S, X3-3.S
- new net BOOT0: R27.1, U1.BOOT0
- new net CRUISE_LAMP_OUT_PB15: Q1.G, R22.1, U1.PB15
- new net D_IN: C7.+, R12.2, X3-2.S
- new net D_IN_PA8: D4.C, R12.1, R13.1, U1.PA8
- new net IDLE_IN: C6.+, R10.1, X4-5.S
- new net IDLE_IN_PB14: D6.C, R10.2, R11.2, U1.PB14
- new net M0: M0.P, X2-1.S
- new net M1: M1.P, X2-2.S
- new net N$15: R16.2, R17.1
- new net N$18: U1.PB5
- new net N$2: C9.1, Q4.2, U1.PD0-OSC_IN
- new net N$20: U1.PB3
- new net N$25: U1.PA1
- new net N$26: U1.PA2
- new net N$28: U1.PA4
- new net N$29: U1.PA6
- new net N$3: C10.2, Q4.1, U1.PD1-OSC_OUT
- new net N$30: U1.PA5
- new net N$32: Q1.D, X3-4.S
- new net N$35: Q2.D, X3-5.S
- new net N$4: D1.C, R2.2, R5.1, T2.B
- new net N$41: U1.PA15
- new net N$6: D2.C, R1.2, T1.B
- new net N$7: J1.2, R27.2
- new net N$9: C11.1, S1.2
- new net OD_IN_L: C5.+, R8.2, X3-1.S
- new net OD_IN_LIGHT_PB12: D5.C, R8.1, R9.1, U1.PB12
- new net OD_OUT_BUTTON_PB13: Q2.G, R23.1, U1.PB13
- new net RST: C11.2, S1.1, U1.NRST
- new net STOP_IN_PA3: D3.C, R6.2, R7.2, U1.PA3
- new net SW_IN: C8.+, R18.1, X1-2.S
- net GND: now also C10.1, C12.1, C13.1, C14.1, C15.1, C16.1, C17.1, C18.1, C19.1, C2.2, C3.-, C5.-, C6.-, C7.-, C8.-, C9.2, D1.A, D2.A, D3.A, D4.A, D5.A, D6.A, D7.A, D8.A, J1.1, Q1.S, Q2.S, Q3.S, R11.1, R13.2, R15.2, R17.2, R21.2, R22.2, R23.2, R24.2, R5.2, R7.1, R9.2, X1-1.S, X4-6.S; no longer C2.-, C3.2, R10.1, R12.1, R2.1, R4.1, R6.1, R8.1, T3.E
- net N$1: now also Q3.D, X2-4.S; no longer R11.1, R12.2, T1.B
- net PB2_OUT_SOLENOID: now also Q3.G, R24.1, U1.PB2; no longer U1.PA8
- net RPM_EXTI11: now also R4.1, T2.C; no longer R13.1, T1.C
- net RPM_IN: now also R2.1, X4-2.S; no longer R11.2
- net SCL: now also R25.2, U1.PB6; no longer R16.1
- net SDA: now also R26.2, U1.PB7; no longer R17.1
- net SPD_IN: now also C2.1, R1.1, X4-3.S; no longer C3.1, R5.2
- net STOP_IN: now also C4.+, R6.1, X4-4.S; no longer C2.+, R7.2
- net SWITCH_ADC: now also D7.C, R18.2, R19.1
- net TIM3_CH2_SPD: now also R3.1, T1.C; no longer R15.1, R5.1, R6.2, T3.B, T3.C
- net TPS_ADC: now also C3.+, D8.C, R20.2, R21.1; no longer R1.1, R2.2
- net TPS_IN: now also R20.1, X4-1.S; no longer C4.+, R1.2
- net VCC: now also C12.2, C13.2, C14.2, C15.2, C16.2, C17.2, C18.2, C19.2, J1.3, R19.2, R25.1, R26.1, R3.2, R4.2, U1.VDDA, U1.VDD_1, U1.VDD_2, U1.VDD_3; no longer R13.2, R14.2, R15.2, R16.2, R17.2
- net VNH2_SP30_CS: now also PAD4.P, R16.1; no longer R10.2, R9.1
- net VNH2_SP30_EN: now also PAD3.P, R14.2, R15.1; no longer R3.1, R4.2
- net VNH2_SP30_EN_IN: now also R14.1; no longer R3.2
- net VNH2_SP30_INA: now also PAD1.P
- net VNH2_SP30_INB: now also PAD2.P
- net VNH2_SP30_PWM: now also PAD5.P
Other:
- note removed: "15v max"
- note removed: "5v max"
- moved on the sheet: C1, C4, IC1, R1, R10, R11, R12, R13, R14, R15, R16, R17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

Commit message: работа над схемой
Parts:
- removed PAD1, PAD2, PAD3, PAD4, PAD5: (no value), wirepad:2,54/1,0
- added CS, EN, INA, INB, PWM: (no value), wirepad:2,54/1,0
- added IC2: 7805T, linear:7805T
- added IC3: LD117AS33TR, v-reg:LD117AS33TR
- added Q5, Q6, Q7: BSS138, m-pad-2.1:BSS138
- added R28, R29, R30, R32, R33: 10K, resistor:R-EU_R0805
- added R31: 510, resistor:R-EU_R0805
Connections:
- removed net N$15: R16.2, R17.1
- new net +5V: IC2.VO, IC3.IN, R31.1, R32.1, R33.1
- new net N$10: INA.P, Q5.D, R33.2
- new net N$5: PWM.P, Q7.D, R31.2
- new net N$8: INB.P, Q6.D, R32.2
- new net VNH2_SP30_CS_IN: CS.P, R16.1
- net +12V: now also IC2.VI
- net GND: now also IC2.GND, IC3.ADJ
- net VCC: now also IC3.OUT, Q5.G, Q6.G, Q7.G, R28.2, R29.1, R30.2
- net VNH2_SP30_CS: now also R16.2, R17.1; no longer PAD4.P, R16.1
- net VNH2_SP30_EN: no longer PAD3.P
- net VNH2_SP30_EN_IN: now also EN.P
- net VNH2_SP30_INA: now also Q5.S, R30.1; no longer PAD1.P
- net VNH2_SP30_INB: now also Q6.S, R28.1; no longer PAD2.P
- net VNH2_SP30_PWM: now also Q7.S, R29.2; no longer PAD5.P

Commit message: схема
Parts:
- added +12V4A, +5V, GND: (no value), wirepad:2,54/1,0
- added ARMED, D_IN, IDLE, OD_IN, OD_OUT, RPM, SL, SPD, STOP, VCC: (no value), led:LEDCHIP-LED0805
- added C20: 470uF, rcl:CPOL-EUG
- added C21, C23, C25: 100nf, rcl:C-EUC0805
- added C22, C24: 220uF, rcl:CPOL-EUCT6032
- added F1: 500mA, m-pad-2.1:FUSEC
- added F2: 2000mA, m-pad-2.1:FUSEC
- added F3: 4000mA, m-pad-2.1:FUSEC
- added JP1: (no value), jumper:JP10Q
- added R34, R35: 200, resistor:R-EU_R0805
- added R36, R37, R38, R39, R40, R41, R42, R43, R44, R45: 510, resistor:R-EU_R0805
- added U$1: (no value), my:INDUCTORCD43-3D
- added X5: SWD, Rembrandt Electronics - JST XH Connectors v1-0:JST-XH-06-PIN-LONG-PAD
- added X6: I2C, Rembrandt Electronics - JST XH Connectors v1-0:JST-XH-04-PIN-LONG-PAD
- added X7: JST-XH-06-PIN-LONG-PAD, Rembrandt Electronics - JST XH Connectors v1-0:JST-XH-06-PIN-LONG-PAD
- C1, C10, C11, C12, C13, C14, C15, C16, C17, C18, C19, C2, C9: device rcl:C-EUC0805 -> rcl:C-EUC0805K
- C3: value 5uF -> 100nf; device rcl:CPOL-EUCT6032 -> rcl:C-EUC0805K
- C4, C5, C7: value 10uF -> 100nf; device rcl:CPOL-EUCT6032 -> rcl:C-EUC0805K
- C6, C8: value 1uF -> 100nf; device rcl:CPOL-EUCT6032 -> rcl:C-EUC0805K
- Q4: device crystal:CRYSTALSM49 -> crystal-geyer_V1_0:KX-9B
Connections:
- new net +12V2A: F2.2
- new net +12V4A: +12V4A.P, F3.2, X2-3.S
- new net +12V_FUSED: C20.+, C21.2, IC2.VI, U$1.P$2
- new net N$11: R34.1, X6-3.S
- new net N$12: R35.1, X6-4.S
- new net N$13: F1.2, U$1.P$1
- new net N$14: JP1.20, R36.2
- new net N$15: R36.1, RPM.A
- new net N$16: R37.1, SPD.A
- new net N$17: R38.1, STOP.A
- new net N$19: OD_IN.A, R39.1
- new net N$21: D_IN.A, R40.1
- new net N$22: IDLE.A, R41.1
- new net N$23: R42.1, VCC.A
- new net N$24: ARMED.A, R43.1
- new net N$27: JP1.18, R37.2
- new net N$31: JP1.16, R38.2
- new net N$33: JP1.14, R39.2
- new net N$42: JP1.8, R42.2
- new net N$43: JP1.6, R43.2
- new net N$44: OD_OUT.A, R44.1
- new net N$45: R45.1, SL.A
- new net N$46: JP1.4, R44.2
- new net N$47: JP1.2, R45.2
- new net SWDCLK: U1.PA14, X5-4.S
- new net SWDIO: U1.PA13, X5-3.S
- net +12V: now also F1.1, F2.1, F3.1, X7-4.S, X7-5.S, X7-6.S; no longer IC2.VI, X2-3.S, X3-3.S
- net +5V: now also +5V.P, C22.+, C23.2
- net CRUISE_LAMP_OUT_PB15: now also JP1.7
- net D_IN: now also C7.1; no longer C7.+
- net D_IN_PA8: now also JP1.5
- net GND: now also ARMED.C, C20.-, C21.1, C22.-, C23.1, C24.-, C25.1, C3.2, C4.2, C5.2, C6.2, C7.2, C8.2, D_IN.C, GND.P, IDLE.C, OD_IN.C, OD_OUT.C, RPM.C, SL.C, SPD.C, STOP.C, U1.VSSA, U1.VSS_1, U1.VSS_2, U1.VSS_3, VCC.C, X5-1.S, X6-1.S, X7-1.S, X7-2.S, X7-3.S; no longer C3.-, C4.-, C5.-, C6.-, C7.-, C8.-
- net IDLE_IN: now also C6.1; no longer C6.+
- net IDLE_IN_PB14: now also JP1.9
- net N$39: now also JP1.12, R40.2; no longer U1.PA13
- net N$40: now also JP1.10, R41.2; no longer U1.PA14
- net OD_IN_L: now also C5.1; no longer C5.+
- net OD_IN_LIGHT_PB12: now also JP1.13
- net OD_OUT_BUTTON_PB13: now also JP1.11
- net PB2_OUT_SOLENOID: now also JP1.17
- net RPM_EXTI11: now also JP1.15
- net SCL: now also R35.2
- net SDA: now also R34.2
- net STOP_IN: now also C4.1; no longer C4.+
- net STOP_IN_PA3: now also JP1.19
- net SW_IN: now also C8.1; no longer C8.+
- net TIM3_CH2_SPD: now also JP1.1
- net TPS_ADC: now also C3.1; no longer C3.+
- net VCC: now also C24.+, C25.2, JP1.3, X5-2.S, X6-2.S
Other:
- moved on the sheet: IC2

Commit message: схема+проверка работы мотора
какой то косяк с шимом. Наверное зря удалил подтягивающий резистор. Нормально работает только на частоте до 1кгц
Parts:
- removed +12V4A, +5V, CS, EN, GND, INA, INB, M0, M1, PWM: (no value), wirepad:2,54/1,0
- removed ARMED, D_IN, IDLE, OD_IN, OD_OUT, RPM, SL, SPD, STOP, VCC: (no value), led:LEDCHIP-LED0805
- removed C21: 100nf, rcl:C-EUC0805
- removed IC2: 7805T, linear:7805T
- removed JP1: (no value), jumper:JP10Q
- removed Q5, Q6, Q7: BSS138, m-pad-2.1:BSS138
- removed R14, R16, R28, R29, R30, R32, R33: 10K, resistor:R-EU_R0805
- removed R15, R17: 6.8K, resistor:R-EU_R0805
- removed R31, R36, R37, R38, R39, R40, R41, R42, R43, R44, R45: 510, resistor:R-EU_R0805
- added D9: (no value), eagle-ltspice:SCHOTTKY-DIODESMC
- added F4: 500mA, m-pad-2.1:FUSEC
- added TB1: TB6612FNG, TB6612FNG:TB6612FNG
- added U$6: MP1584, MP1584-dc-brick:MP1584
- F3: value 4000mA -> 2000mA
Connections:
- removed net +12V2A: F2.2
- removed net +12V4A: +12V4A.P, F3.2, X2-3.S
- removed net +12V_FUSED: C20.+, C21.2, IC2.VI, U$1.P$2
- removed net N$10: INA.P, Q5.D, R33.2
- removed net N$14: JP1.20, R36.2
- removed net N$15: R36.1, RPM.A
- removed net N$16: R37.1, SPD.A
- removed net N$17: R38.1, STOP.A
- removed net N$19: OD_IN.A, R39.1
- removed net N$21: D_IN.A, R40.1
- removed net N$23: R42.1, VCC.A
- removed net N$24: ARMED.A, R43.1
- removed net N$27: JP1.18, R37.2
- removed net N$31: JP1.16, R38.2
- removed net N$33: JP1.14, R39.2
- removed net N$39: JP1.12, R40.2
- removed net N$40: JP1.10, R41.2
- removed net N$42: JP1.8, R42.2
- removed net N$43: JP1.6, R43.2
- removed net N$44: OD_OUT.A, R44.1
- removed net N$45: R45.1, SL.A
- removed net N$46: JP1.4, R44.2
- removed net N$47: JP1.2, R45.2
- removed net N$8: INB.P, Q6.D, R32.2
- removed net VNH2_SP30_CS: R16.2, R17.1, U1.PA7
- removed net VNH2_SP30_CS_IN: CS.P, R16.1
- removed net VNH2_SP30_EN_IN: EN.P, R14.1
- new net +12V2A_MOTOR: F3.2, TB1.VM
- new net +12V2A_SOLENOID: F2.2, X2-3.S
- new net 12V_500MA_SENSORS: F1.2
- net +12V: now also U$1.P$1; no longer F1.1, F3.1
- net +5V: now also F4.2; no longer +5V.P, IC2.VO, R31.1, R32.1, R33.1
- net CRUISE_LAMP_OUT_PB15: no longer JP1.7
- net D_IN_PA8: no longer JP1.5
- net GND: now also TB1.GND1, TB1.GND2, TB1.GND3, U$6.VIN-, U$6.VOUT-; no longer ARMED.C, C21.1, D_IN.C, GND.P, IC2.GND, IDLE.C, OD_IN.C, OD_OUT.C, R15.2, R17.2, RPM.C, SL.C, SPD.C, STOP.C, VCC.C
- net IDLE_IN_PB14: no longer JP1.9
- net M0: now also TB1.A2, TB1.B2; no longer M0.P
- net M1: now also TB1.A1, TB1.B1; no longer M1.P
- net N$13: now also D9.C, U$1.P$2; no longer F1.2, U$1.P$1
- net N$22: now also C20.+, D9.A, F1.1, U$6.VIN+; no longer IDLE.A, R41.1
- net N$5: now also F3.1, F4.1, U$6.VOUT+; no longer PWM.P, Q7.D, R31.2
- net OD_IN_LIGHT_PB12: no longer JP1.13
- net OD_OUT_BUTTON_PB13: no longer JP1.11
- net PB2_OUT_SOLENOID: no longer JP1.17
- net RPM_EXTI11: no longer JP1.15
- net STOP_IN_PA3: no longer JP1.19
- net TIM3_CH2_SPD: no longer JP1.1
- net VCC: now also TB1.VCC; no longer JP1.3, Q5.G, Q6.G, Q7.G, R28.2, R29.1, R30.2
- net VNH2_SP30_EN: now also TB1.STBY; no longer R14.2, R15.1
- net VNH2_SP30_INA: now also TB1.AIN1, TB1.BIN1; no longer Q5.S, R30.1
- net VNH2_SP30_INB: now also TB1.AIN2, TB1.BIN2; no longer Q6.S, R28.1
- net VNH2_SP30_PWM: now also TB1.PWMA, TB1.PWMB; no longer Q7.S, R29.2
Other:
- moved on the sheet: C20, F1, F2, F3, Q3, R24, X2-1, X2-2, X2-3, X2-4, X7-1, X7-2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

Commit message: PWM+PID
Заработал нормально Pwm 20khz
Заработал вменяемо PID
Parts:
- added R14, R15, R16: 200, resistor:R-EU_R0805
- Q1, Q2, Q3: value BSS138 -> AO4300
Connections:
- net N$18 renamed PB5_OUT_SOLENOID
- removed net N$20: U1.PB3
- removed net PB2_OUT_SOLENOID: Q3.G, R24.1, U1.PB2
- removed net VNH2_SP30_EN: TB1.STBY, U1.PB10
- new net N$10: Q1.G, R15.2, R22.1
- new net N$14: Q2.G, R16.2, R23.1
- new net N$8: Q3.G, R14.2, R24.1
- new net PB10_OUT_SOLENOID: R14.1, U1.PB10
- new net TB6612FNG_STB: TB1.STBY, U1.PB2
- net CRUISE_LAMP_OUT_PB15: now also R15.1; no longer Q1.G, R22.1
- net D_IN: now also X3-1.S; no longer X3-2.S
- net N$32: now also X3-5.S; no longer X3-4.S
- net N$35: now also X3-4.S; no longer X3-5.S
- net OD_IN_L: now also X3-2.S; no longer X3-1.S
- net OD_OUT_BUTTON_PB13: now also R16.1; no longer Q2.G, R23.1
- net SCL: now also R34.2; no longer R35.2
- net SDA: now also R35.2; no longer R34.2
Other:
- moved on the sheet: Q2, R23

Commit message: добавлен функционал тюна пидов
Parts:
- added CRUISE, D_IN, IDLE, LED11, LED12, OD_IN, OD_OUT, RPM, SPD: (no value), led:LEDCHIP-LED0805
- added RN1, RN2, RN3: (no value), resistor-dil:4R-N0603-ARV
- added SLD, STOP, VCC: (no value), led:LEDCHIPLED_0805
Connections:
- new net N$15: RN1B.1, RPM.A
- new net N$16: RN1A.1, VCC.A
- new net N$17: RN1C.1, SPD.A
- new net N$18: CRUISE.A, RN1D.1
- new net N$19: RN2A.1, STOP.A
- new net N$20: OD_IN.A, RN2B.1
- new net N$21: IDLE.A, RN2C.1
- new net N$23: OD_OUT.A, RN2D.1
- new net N$24: RN3A.1, SLD.A
- new net N$27: D_IN.A, RN3B.1
- new net N$31: LED11.A, RN3C.1
- new net N$33: LED12.A, RN3D.1
- net CRUISE_LAMP_OUT_PB15: now also RN1D.2
- net D_IN_PA8: now also RN3B.2
- net GND: now also CRUISE.C, D_IN.C, IDLE.C, LED11.C, LED12.C, OD_IN.C, OD_OUT.C, RPM.C, SLD.C, SPD.C, STOP.C, VCC.C
- net IDLE_IN_PB14: now also RN2C.2
- net OD_IN_LIGHT_PB12: now also RN2B.2
- net OD_OUT_BUTTON_PB13: now also RN2D.2
- net PB10_OUT_SOLENOID: now also RN3A.2
- net RPM_EXTI11: now also RN1B.2
- net STOP_IN_PA3: now also RN2A.2
- net TIM3_CH2_SPD: now also RN1C.2
- net VCC: now also RN1A.2

Commit message: измененние схемы
Parts:
- removed CRUISE, D_IN, IDLE, LED11, LED12, OD_IN, OD_OUT, RPM, SPD: (no value), led:LEDCHIP-LED0805
- removed R3: 4.7K, resistor:R-EU_R0805
- removed RN1, RN2, RN3: (no value), resistor-dil:4R-N0603-ARV
- removed SLD, STOP, VCC: (no value), led:LEDCHIPLED_0805
- removed T1, T2: (no value), transistor-neu-to92:MMBT4401LT1-NPN-SOT23-BEC
- R11, R13, R7, R9: value 3.3K -> 3K
- renumbered X1 to SW, X2 to MOT, X3 to IO1, X7 to PWR
Connections:
- removed net N$15: RN1B.1, RPM.A
- removed net N$16: RN1A.1, VCC.A
- removed net N$17: RN1C.1, SPD.A
- removed net N$18: CRUISE.A, RN1D.1
- removed net N$19: RN2A.1, STOP.A
- removed net N$20: OD_IN.A, RN2B.1
- removed net N$21: IDLE.A, RN2C.1
- removed net N$23: OD_OUT.A, RN2D.1
- removed net N$24: RN3A.1, SLD.A
- removed net N$27: D_IN.A, RN3B.1
- removed net N$31: LED11.A, RN3C.1
- removed net N$33: LED12.A, RN3D.1
- removed net N$4: D1.C, R2.2, R5.1, T2.B
- removed net N$6: D2.C, R1.2, T1.B
- net CRUISE_LAMP_OUT_PB15: no longer RN1D.2
- net D_IN_PA8: no longer RN3B.2
- net GND: now also R4.2; no longer CRUISE.C, D_IN.C, IDLE.C, LED11.C, LED12.C, OD_IN.C, OD_OUT.C, RPM.C, SLD.C, SPD.C, STOP.C, T1.E, T2.E, VCC.C
- net IDLE_IN_PB14: no longer RN2C.2
- net OD_IN_LIGHT_PB12: no longer RN2B.2
- net OD_OUT_BUTTON_PB13: no longer RN2D.2
- net PB10_OUT_SOLENOID: no longer RN3A.2
- net RPM_EXTI11: now also D1.C, R2.2, R5.1; no longer R4.1, RN1B.2, T2.C
- net STOP_IN_PA3: no longer RN2A.2
- net TIM3_CH2_SPD: now also D2.C, R1.2, R4.1; no longer R3.1, RN1C.2, T1.C
- net VCC: no longer R3.2, R4.2, RN1A.2
Other:
- note added: "10k+6,8k = 5V"
- note added: "12V max 5V tolerant"
- note added: "5V max 3V3 tolerant"
- note added: "8V max 5V tolerant"
- moved on the sheet: C1, C2, D1, D2, R1, R2, R4, R5

Commit message: работа со схемой
Parts:
- removed F1: 500mA, m-pad-2.1:FUSEC
- added C21: 470uF, rcl:CPOL-EUG
- added CTS, PA15_ADC, PA1_ADC, PA2_ADC, PA4_ADC, PA5_ADC, PA6_ADC, PA7_ADC, PB3, PB5, PC13, RTC-14, RTC-15, RTS: TPTP09R, testpad:TPTP09R
- IO1: value JST-XH-05-PIN-LONG-PAD -> JST-XH-04-PIN-LONG-PAD; device Rembrandt Electronics - JST XH Connectors v1-0:JST-XH-05-PIN-LONG-PAD -> Rembrandt Electronics - JST XH Connectors v1-0:JST-XH-04-PIN-LONG-PAD
- renumbered X4 to IO2
Connections:
- removed net 12V_500MA_SENSORS: F1.2
- removed net N$22: C20.+, D9.A, F1.1, U$6.VIN+
- removed net N$34: U1.PA9
- removed net N$36: U1.PA10
- removed net N$41: U1.PA15
- removed net PB5_OUT_SOLENOID: U1.PB5
- new net N$15: PC13.TP, U1.PC13-TAMPER-RTC
- new net N$16: RTC-14.TP, U1.PC14-OSC32_IN
- new net N$17: RTC-15.TP, U1.PC15-OSC32_OUT
- new net N$18: C20.+, D9.A, U$6.VIN+
- new net N$4: PA7_ADC.TP, U1.PA7
- new net N$6: PB3.TP, U1.PB3
- new net PA15_ADC: PA15_ADC.TP, U1.PA15
- new net PB5: PB5.TP, U1.PB5
- new net RX: U1.PA10, X5-5.S
- new net TX: U1.PA9, X5-6.S
- net GND: now also C21.-; no longer IO2-6.S
- net N$25: now also PA1_ADC.TP
- net N$26: now also PA2_ADC.TP
- net N$28: now also PA4_ADC.TP
- net N$29: now also PA6_ADC.TP
- net N$30: now also PA5_ADC.TP
- net N$32: now also IO1-4.S; no longer IO1-5.S
- net N$35: now also IO1-3.S; no longer IO1-4.S
- net N$37: now also CTS.TP
- net N$38: now also RTS.TP
- net N$5: now also C21.+
Other:
- moved on the sheet: IO1-1, IO1-2, IO1-3, IO1-4
