File: cruise/cruise.sch (EAGLE design)
At the start: 97 parts, among them IC1 24C04ASM, IC3 LD117AS33TR, Q1 AO4300, Q2 AO4300, Q3 AO4300, Q4 8MHz, U1 STM32F103CBT6, X5 SWD, X6 I2C

Commit message: еще схема
Parts:
- removed U$1: (no value), my:INDUCTORCD43-3D
- IO1: value JST-XH-04-PIN-LONG-PAD -> JST-XH-04-PIN-ROUND-PAD; device Rembrandt Electronics - JST XH Connectors v1-0:JST-XH-04-PIN-LONG-PAD -> Rembrandt Electronics - JST XH Connectors v1-0:JST-XH-04-PIN-ROUND-PAD
- IO2: value JST-XH-06-PIN-LONG-PAD -> JST-XH-06-PIN-ROUND-PAD; device Rembrandt Electronics - JST XH Connectors v1-0:JST-XH-06-PIN-LONG-PAD -> Rembrandt Electronics - JST XH Connectors v1-0:JST-XH-06-PIN-ROUND-PAD
- SW: value JST-XH-02-PIN-LONG-PAD -> JST-XH-02-PIN-ROUND-PAD; device Rembrandt Electronics - JST XH Connectors v1-0:JST-XH-02-PIN-LONG-PAD -> Rembrandt Electronics - JST XH Connectors v1-0:JST-XH-02-PIN-ROUND-PAD
- X5: device Rembrandt Electronics - JST XH Connectors v1-0:JST-XH-06-PIN-LONG-PAD -> Rembrandt Electronics - JST XH Connectors v1-0:JST-XH-06-PIN-ROUND-PAD
- X6: device Rembrandt Electronics - JST XH Connectors v1-0:JST-XH-04-PIN-LONG-PAD -> Rembrandt Electronics - JST XH Connectors v1-0:JST-XH-04-PIN-ROUND-PAD
Connections:
- removed net N$13: D9.C, U$1.P$2
- net +12V: now also D9.C; no longer U$1.P$1
Other:
- moved on the sheet: C20, D9, F3

Commit message: ds
Parts:
- removed C22: 220uF, rcl:CPOL-EUCT6032
- C10: device rcl:C-EUC0805K -> rcl:C-EUC0603
- C15: value 10uF -> 100nf
- C24: value 220uF -> 100uF; device rcl:CPOL-EUCT6032 -> resistor:C-EUC1210
- C9: device rcl:C-EUC0805K -> resistor:C-EUC0603
- IC1: value 24C04ASM -> 24C04ASN; device microchip:24C04ASM -> microchip:24C04ASN
Connections:
- net +5V: no longer C22.+
- net GND: now also C24.2; no longer C22.-, C24.-
- net VCC: now also C24.1; no longer C24.+
Changed lines of the file:
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@@
 <?xml version="1.0" encoding="utf-8"?>
 <!DOCTYPE eagle SYSTEM "eagle.dtd">
-<eagle version="9.2.2">
+<eagle version="9.3.1">
 <drawing>
 <settings>
@@
 </classes>
 <parts>
-<part name="IC1" library="microchip" library_urn="urn:adsk.eagle:library:294" deviceset="24C*" device="SM" package3d_urn="urn:adsk.eagle:package:20798/1" technology="04A"/>
+<part name="IC1" library="microchip" library_urn="urn:adsk.eagle:library:294" deviceset="24C*" device="SN" package3d_urn="urn:adsk.eagle:package:20804/2" technology="04A" value="24C04ASN"/>
 <part name="R1" library="resistor" library_urn="urn:adsk.eagle:library:348" deviceset="R-EU_" device="R0805" package3d_urn="urn:adsk.eagle:package:23553/2" value="10K"/>
 <part name="R2" library="resistor" library_urn="urn:adsk.eagle:library:348" deviceset="R-EU_" device="R0805" package3d_urn="urn:adsk.eagle:package:23553/2" value="10K"/>
@@
 <part name="P+3" library="supply1" library_urn="urn:adsk.eagle:library:371" deviceset="VCC" device=""/>
 <part name="Q4" library="crystal-geyer_V1_0" library_urn="urn:adsk.eagle:library:203" deviceset="KX" device="-9B" package3d_urn="urn:adsk.eagle:package:11930/1" value="8MHz"/>
-<part name="C9" library="rcl" library_urn="urn:adsk.eagle:library:334" deviceset="C-EU" device="C0805K" package3d_urn="urn:adsk.eagle:package:23681/2" value="20pf"/>
-<part name="C10" library="rcl" library_urn="urn:adsk.eagle:library:334" deviceset="C-EU" device="C0805K" package3d_urn="urn:adsk.eagle:package:23681/2" value="20pf"/>
+<part name="C9" library="resistor" library_urn="urn:adsk.eagle:library:348" deviceset="C-EU" device="C0603" package3d_urn="urn:adsk.eagle:package:23616/2" value="20pf"/>
+<part name="C10" library="rcl" library_urn="urn:adsk.eagle:library:334" deviceset="C-EU" device="C0603" package3d_urn="urn:adsk.eagle:package:23616/2" value="20pf"/>
 <part name="J1" library="jumper" library_urn="urn:adsk.eagle:library:252" deviceset="J2" device="X2MM" package3d_urn="urn:adsk.eagle:package:15506/1"/>
 <part name="R27" library="resistor" library_urn="urn:adsk.eagle:library:348" deviceset="R-EU_" device="R0805" package3d_urn="urn:adsk.eagle:package:23553/2" value="10K"/>
@@
 <part name="P+6" library="supply1" library_urn="urn:adsk.eagle:library:371" deviceset="VCC" device=""/>
 <part name="C14" library="rcl" library_urn="urn:adsk.eagle:library:334" deviceset="C-EU" device="C0805K" package3d_urn="urn:adsk.eagle:package:23681/2" value="100nf"/>
-<part name="C15" library="rcl" library_urn="urn:adsk.eagle:library:334" deviceset="C-EU" device="C0805K" package3d_urn="urn:adsk.eagle:package:23681/2" value="10uF"/>
+<part name="C15" library="rcl" library_urn="urn:adsk.eagle:library:334" deviceset="C-EU" device="C0805K" package3d_urn="urn:adsk.eagle:package:23681/2" value="100nf"/>
 <part name="C16" library="rcl" library_urn="urn:adsk.eagle:library:334" deviceset="C-EU" device="C0805K" package3d_urn="urn:adsk.eagle:package:23681/2" value="100nf"/>
 <part name="C17" library="rcl" library_urn="urn:adsk.eagle:library:334" deviceset="C-EU" device="C0805K" package3d_urn="urn:adsk.eagle:package:23681/2" value="100nf"/>
@@
 <part name="GND17" library="supply1" library_urn="urn:adsk.eagle:library:371" deviceset="GND" device=""/>
 <part name="C20" library="rcl" library_urn="urn:adsk.eagle:library:334" deviceset="CPOL-EU" device="G" package3d_urn="urn:adsk.eagle:package:23427/2" value="470uF"/>
-<part name="C22" library="rcl" library_urn="urn:adsk.eagle:library:334" deviceset="CPOL-EU" device="CT6032" package3d_urn="urn:adsk.eagle:package:23305/2" value="220uF"/>
 <part name="C23" library="rcl" library_urn="urn:adsk.eagle:library:334" deviceset="C-EU" device="C0805" package3d_urn="urn:adsk.eagle:package:23617/2" value="100nf"/>
-<part name="C24" library="rcl" library_urn="urn:adsk.eagle:library:334" deviceset="CPOL-EU" device="CT6032" package3d_urn="urn:adsk.eagle:package:23305/2" value="220uF"/>
+<part name="C24" library="resistor" library_urn="urn:adsk.eagle:library:348" deviceset="C-EU" device="C1210" package3d_urn="urn:adsk.eagle:package:23619/2" value="100uF"/>
 <part name="C25" library="rcl" library_urn="urn:adsk.eagle:library:334" deviceset="C-EU" device="C0805" package3d_urn="urn:adsk.eagle:package:23617/2" value="100nf"/>
 <part name="F2" library="m-pad-2.1" deviceset="FUSE" device="C" value="2000mA"/>
@@
 <attribute name="VALUE" x="-285.877" y="246.8626" size="1.778" layer="96"/>
 </instance>
-<instance part="C22" gate="G$1" x="-185.42" y="246.38" smashed="yes">
-<attribute name="NAME" x="-184.277" y="246.8626" size="1.778" layer="95"/>
-<attribute name="VALUE" x="-184.277" y="241.7826" size="1.778" layer="96"/>
-</instance>
 <instance part="C23" gate="G$1" x="-170.18" y="243.84" smashed="yes" rot="R180">
 <attribute name="NAME" x="-171.704" y="243.459" size="1.778" layer="95" rot="R180"/>
@@
 </instance>
 <instance part="C21" gate="G$1" x="-210.82" y="248.92" smashed="yes">
-<attribute name="NAME" x="-240.157" y="249.4026" size="1.778" layer="95"/>
-<attribute name="VALUE" x="-242.697" y="244.3226" size="1.778" layer="96"/>
+<attribute name="NAME" x="-217.297" y="244.3226" size="1.778" layer="95"/>
+<attribute name="VALUE" x="-219.837" y="241.7826" size="1.778" layer="96"/>
 </instance>
 <instance part="IO1" gate="-1" x="86.36" y="86.36" smashed="yes">
@@
 <segment>
 <pinref part="IC3" gate="G$1" pin="ADJ"/>
-<wire x1="-185.42" y1="231.14" x2="-170.18" y2="231.14" width="0.1524" layer="91"/>
 <wire x1="-170.18" y1="231.14" x2="-160.02" y2="231.14" width="0.1524" layer="91"/>
 <wire x1="-160.02" y1="231.14" x2="-160.02" y2="243.84" width="0.1524" layer="91"/>
-<pinref part="C22" gate="G$1" pin="-"/>
-<wire x1="-185.42" y1="241.3" x2="-185.42" y2="231.14" width="0.1524" layer="91"/>
 <pinref part="C23" gate="G$1" pin="1"/>
 <wire x1="-170.18" y1="241.3" x2="-170.18" y2="231.14" width="0.1524" layer="91"/>
 <junction x="-170.18" y="231.14"/>
-<pinref part="C24" gate="G$1" pin="-"/>
+<pinref part="C24" gate="G$1" pin="2"/>
 <wire x1="-149.86" y1="241.3" x2="-149.86" y2="231.14" width="0.1524" layer="91"/>
 <wire x1="-149.86" y1="231.14" x2="-160.02" y2="231.14" width="0.1524" layer="91"/>
@@
 <wire x1="-228.6" y1="246.38" x2="-228.6" y2="231.14" width="0.1524" layer="91"/>
 <wire x1="-228.6" y1="231.14" x2="-210.82" y2="231.14" width="0.1524" layer="91"/>
-<junction x="-185.42" y="231.14"/>
 <pinref part="C21" gate="G$1" pin="-"/>
-<wire x1="-210.82" y1="231.14" x2="-185.42" y2="231.14" width="0.1524" layer="91"/>
+<wire x1="-210.82" y1="231.14" x2="-170.18" y2="231.14" width="0.1524" layer="91"/>
 <wire x1="-210.82" y1="243.84" x2="-210.82" y2="231.14" width="0.1524" layer="91"/>
 <junction x="-210.82" y="231.14"/>
@@
 <wire x1="-152.4" y1="251.46" x2="-149.86" y2="251.46" width="0.1524" layer="91"/>
 <label x="-139.7" y="251.46" size="1.778" layer="95"/>
-<pinref part="C24" gate="G$1" pin="+"/>
+<pinref part="C24" gate="G$1" pin="1"/>
 <wire x1="-149.86" y1="251.46" x2="-134.62" y2="251.46" width="0.1524" layer="91"/>
 <wire x1="-134.62" y1="251.46" x2="-127" y2="251.46" width="0.1524" layer="91"/>
@@
 <wire x1="-170.18" y1="251.46" x2="-170.18" y2="248.92" width="0.1524" layer="91"/>
 <junction x="-170.18" y="251.46"/>
-<pinref part="C22" gate="G$1" pin="+"/>
-<wire x1="-185.42" y1="251.46" x2="-185.42" y2="248.92" width="0.1524" layer="91"/>
-<wire x1="-185.42" y1="251.46" x2="-170.18" y2="251.46" width="0.1524" layer="91"/>
+<wire x1="-195.58" y1="251.46" x2="-170.18" y2="251.46" width="0.1524" layer="91"/>
 <pinref part="F4" gate="G$1" pin="2"/>
-<wire x1="-195.58" y1="251.46" x2="-185.42" y2="251.46" width="0.1524" layer="91"/>
-<junction x="-185.42" y="251.46"/>
-</segment>
-</net>
+</segment>
+</net>
