File: cruise/cruise.brd (EAGLE design)
At the start: 75.2 x 58.4 mm, 101 parts, among them IC1 24C04ASM, IC3 LD117AS33TR, Q1 AO4300, Q2 AO4300, Q3 AO4300, Q4 8MHz, U1 STM32F103CBT6, X5 SWD, X6 I2C

Commit message: еще схема
Parts:
- removed U$1: (no value), my:DFN450X400X350-2
- IO1: value (none) -> JST-XH-04-PIN-ROUND-PAD; device Rembrandt Electronics - JST XH Connectors v1-0:JST-XH-04-PACKAGE-LONG-PAD -> Rembrandt Electronics - JST XH Connectors v1-0:JST-XH-04-PACKAGE-ROUND-PAD
- IO2: value (none) -> JST-XH-06-PIN-ROUND-PAD; device Rembrandt Electronics - JST XH Connectors v1-0:JST-XH-06-PACKAGE-LONG-PAD -> Rembrandt Electronics - JST XH Connectors v1-0:JST-XH-06-PACKAGE-ROUND-PAD
- SW: value (none) -> JST-XH-02-PIN-ROUND-PAD; device Rembrandt Electronics - JST XH Connectors v1-0:JST-XH-02-PACKAGE-LONG-PAD -> Rembrandt Electronics - JST XH Connectors v1-0:JST-XH-02-PACKAGE-ROUND-PAD
- X5: device Rembrandt Electronics - JST XH Connectors v1-0:JST-XH-06-PACKAGE-LONG-PAD -> Rembrandt Electronics - JST XH Connectors v1-0:JST-XH-06-PACKAGE-ROUND-PAD
- X6: device Rembrandt Electronics - JST XH Connectors v1-0:JST-XH-04-PACKAGE-LONG-PAD -> Rembrandt Electronics - JST XH Connectors v1-0:JST-XH-04-PACKAGE-ROUND-PAD
- moved C4 3.31 mm to (59.3, 43.3), turned to 270 degrees
- moved D3 3.31 mm to (59.3, 43.3), turned to 90 degrees
- moved R6 1.80 mm to (61.8, 43.3), turned to 270 degrees
- moved R7 1.80 mm to (61.8, 43.3), turned to 270 degrees
- moved U$3 1.52 mm to (71.0, 54.0)
- moved U$4 1.40 mm to (71.0, 4.00)
- moved PA2_ADC 1.40 mm to (40.1, 26.9)
- moved PA1_ADC 1.40 mm to (40.1, 25.3)
- moved D2 1.27 mm to (64.8, 40.6)
- moved D5 1.27 mm to (64.8, 24.1)
- moved R1 1.27 mm to (64.8, 40.6)
- moved R12 1.27 mm to (64.8, 19.1)
- moved R13 1.27 mm to (64.8, 19.1)
- moved R18 1.27 mm to (64.8, 12.7)
- moved R19 1.27 mm to (64.8, 12.7)
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Connections:
- removed net N$13: D9.A, U$1.2
- net +12V: now also D9.A; no longer U$1.1
Routing:
- net +12V: track 26.1 -> 32.0 mm
- net N$13: track 3.94 -> 0.00 mm
- net STOP_IN_PA3: track 45.7 -> 47.4 mm
- net VNH2_SP30_PWM: track 35.4 -> 36.8 mm
- net VNH2_SP30_INB: track 35.2 -> 36.0 mm
- net D_IN_PA8: track 33.8 -> 34.3 mm

Commit message: Update cruise.brd
Parts:
- moved D8 2.92 mm to (55.5, 35.6)
- moved R21 2.92 mm to (55.5, 35.6)
- moved C4 2.54 mm to (56.8, 43.3)
- moved D3 2.54 mm to (56.8, 43.3)
- moved C3 1.91 mm to (59.1, 35.6)
- moved R20 1.91 mm to (59.1, 35.6)
- moved Q3 1.27 mm to (61.0, 8.89)
- moved R14 1.27 mm to (53.3, 8.89)
- moved R24 1.27 mm to (57.1, 8.89)
- moved R2 1.27 mm to (63.5, 35.6)
- moved R5 1.27 mm to (63.5, 35.6)
- moved R6 1.27 mm to (60.6, 43.3)
- moved R7 1.27 mm to (60.6, 43.3)
- moved R18 0.85 mm to (64.0, 13.1)
- moved R19 0.85 mm to (64.0, 13.1)
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Routing:
- net TPS_IN: track 15.3 -> 17.4 mm
- net OD_IN_LIGHT_PB12: track 31.8 -> 30.3 mm
- net GND: track 119.0 -> 120.4 mm
- net TIM3_CH2_SPD: track 34.4 -> 35.8 mm
- net PB10_OUT_SOLENOID: track 24.5 -> 25.8 mm
- net N$1: track 7.65 -> 6.38 mm
- net RPM_IN: track 7.75 -> 9.02 mm
- net IDLE_IN_PB14: track 35.4 -> 36.5 mm
- net VCC: track 241.6 -> 240.7 mm
- net SW_IN: track 9.81 -> 10.7 mm
- net STOP_IN: track 14.7 -> 15.5 mm
- net D_IN: track 8.96 -> 9.72 mm
- net OD_IN_L: track 8.58 -> 9.34 mm
- net STOP_IN_PA3: track 47.4 -> 46.6 mm
- net TPS_ADC: track 30.0 -> 29.3 mm
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
Commit message: схема
Routing:
- net STOP_IN: track 15.5 -> 17.0 mm

Commit message: ds
Parts:
- removed C22: 220uF, rcl:CT6032
- C10: device rcl:C0805K -> rcl:C0603
- C15: value 10uF -> 100nf
- C24: value 220uF -> 100uF; device rcl:CT6032 -> resistor:C1210
- C9: device rcl:C0805K -> resistor:C0603
- IC1: value 24C04ASM -> 24C04ASN; device microchip:SO-08M -> microchip:SO-08
Connections:
- net +5V: no longer C22.+
- net GND: now also C24.2; no longer C22.-, C24.-
- net VCC: now also C24.1; no longer C24.+
Routing:
- net GND: track 120.4 -> 111.3 mm
- net +5V: track 31.3 -> 22.8 mm
- net VCC: track 240.7 -> 233.8 mm
- net SCL: track 19.8 -> 20.6 mm
